File: Schematics/Kuhglocke_GS/Kuhglocke_GS.kicad_pcb (KiCad board)
At the start: 2 copper layers, 141.6 x 70 mm, 152 parts, among them IC1 P3T1755DPZ, J1 USB_C_Female_USB2_Small, J2 MSD-1-A MicroSD Slot, J4 1S Li-Ion Cell, J5 Speaker, J6 MB_A, J7 MB_B, J8 DB_A, J9 DB_B, Q1 AO3401A, Q2 MMBT3904, Q3 AO3401A, Q4 AO3400A, Q5 MMBT3904, Q6 AO3401A, Q7 AO3400A, SW1 SW_ESP_BOOT_MODE, SW2 SW_ESP_RESET, SW3 SW_DOWN, SW4 SW_ENTER, SW5 SW_UP, SW6 SW_BACK, SW7 PWR, U1 CP2102N-Axx-xQFN28, U10 TPB4056B2X-ES1R, U11 AMS1117-3.3, U12 NAU7802SGI, U2 ESP32-S3-WROOM-1, U3 RFM95W-915S2, U4 ACS70331EOLC, U5 LM66100DCKR, U6 LM66100DCKR, U7 MAX98357AETE_T, U8 TPS63001DRCR, U9 YIC31616GMSGG GPS

Commit message: init commit for migrating avionics comms devices to dedicated repo  - updated datasheets links to local file  - missing exact LoRaSX162 datasheet
Other:
- board text added: "Kuhglocke MB Rev 1.0 (Ground Station Mainboard) QRET May 2024 Kennan Bays Owen Price"
- board text removed: "locked"
