File: Schematics/Handheld_GS/Handheld_GS.kicad_sch (KiCad schematic)
At the start: 152 parts, among them IC1 P3T1755DPZ, J1 MB_A, J2 MB_B, J3 DB_A, J4 DB_B, J5 Speaker, J6 USB_C_Female_USB2_Small, J7 1S Li-Ion Cell, J9 MSD-1-A MicroSD Slot, Q1 AO3401A, Q2 MMBT3904, Q3 MMBT3904, Q4 AO3400A, Q5 AO3400A, Q6 AO3401A, Q7 AO3401A, SW1 SW_ENTER, SW2 SW_BACK, SW3 SW_DOWN, SW4 SW_UP, SW5 SW_ESP_BOOT_MODE, SW6 SW_ESP_RESET, SW7 PWR, U1 CP2102N-Axx-xQFN28, U10 MAX98357AETE_T, U11 RFM95W-915S2, U12 YIC31616GMSGG GPS, U2 ESP32-S3-WROOM-1, U3 TPB4056B2X-ES1R, U4 TPS63001DRCR, U5 LM66100DCKR, U6 LM66100DCKR, U7 NAU7802SGI, U8 ACS70331EOLC, U9 AMS1117-3.3

Commit message: Updated ground station with suggest changes and more, routing done
Parts:
- removed C10, C12, C16, C2, C22, C3, C7: 1uF, Capacitor_SMD:C_0603_1608Metric, symbol Device:C
- removed C11, C17, C18, C21, C24, C26, C29, C30, C4, C9: 0.1uF, Capacitor_SMD:C_0603_1608Metric, symbol Device:C
- removed C14, C15, C20, C23, C25, C28, C5, C6, C8: 10uF, Capacitor_SMD:C_0603_1608Metric, symbol Device:C
- removed C27: 47uF, Capacitor_SMD:C_0805_2012Metric, symbol Device:C
- removed C31: 4.7uF, Capacitor_SMD:C_0603_1608Metric, symbol Device:C
- removed D2, D3: WS2812B, LED_SMD:LED_WS2812B_PLCC4_5.0x5.0mm_P3.2mm, symbol LED:WS2812B
- removed D4: DB_LED (GRN), LED_SMD:LED_0805_2012Metric, symbol Device:LED
- removed D7: INT_PWR_LED (RED), LED_SMD:LED_0805_2012Metric, symbol Device:LED
- removed H5, H6: MountingHole, MountingHole:MountingHole_3.2mm_M3_ISO14580_Pad, symbol Mechanical:MountingHole
- removed IC1: P3T1755DPZ, footprints:P3T1755DPZ, symbol P3T1755DPZ:P3T1755DPZ
- removed J1: MB_A, Connector_PinSocket_1.27mm:PinSocket_2x02_P1.27mm_Vertical, symbol CONN4_LPPB022NFSS-RC_SUL_SOCKET:LPPB022NFSS-RC
- removed J2: MB_B, Connector_PinSocket_1.27mm:PinSocket_2x02_P1.27mm_Vertical, symbol CONN4_LPPB022NFSS-RC_SUL_SOCKET:LPPB022NFSS-RC
- removed J3: DB_A, footprints:HPH2-A-04-UA_PINS, symbol CONN4_LPPB022NFSS-RC_SUL_SOCKET:LPPB022NFSS-RC
- removed J4: DB_B, footprints:HPH2-A-04-UA_PINS, symbol CONN4_LPPB022NFSS-RC_SUL_SOCKET:LPPB022NFSS-RC
- removed J6: USB_C_Female_USB2_Small, footprints:USB_C_DB-108PWB, symbol USB_C:USB_C_Female_USB2_Small
- removed J7: 1S Li-Ion Cell, TerminalBlock_TE-Connectivity:TerminalBlock_TE_282834-2_1x02_P2.54mm_Horizontal, symbol Connector:Screw_Terminal_01x02
- removed J8: ~, Connector_PinHeader_1.27mm:PinHeader_1x08_P1.27mm_Vertical, symbol E-Paper:Generic_E-Paper_Display
- removed J9: MSD-1-A MicroSD Slot, footprints:MicroSD_MSD-1-A, symbol Connector:Micro_SD_Card_Det1
- removed JP1: DB_LED_EN, Jumper:SolderJumper-2_P1.3mm_Bridged_Pad1.0x1.5mm, symbol Jumper:SolderJumper_2_Bridged
- removed JP2: FastCharge, Jumper:SolderJumper-2_P1.3mm_Open_Pad1.0x1.5mm, symbol Jumper:SolderJumper_2_Open
- removed JP4: SPK_DIN, Jumper:SolderJumper-2_P1.3mm_Bridged_Pad1.0x1.5mm, symbol Jumper:SolderJumper_2_Bridged
- removed JP5: Gain, Jumper:SolderJumper-3_P1.3mm_Bridged12_Pad1.0x1.5mm_NumberLabels, symbol Jumper:SolderJumper_3_Bridged12
- removed JP6: DIO2_EN, Jumper:SolderJumper-2_P1.3mm_Open_RoundedPad1.0x1.5mm, symbol Jumper:SolderJumper_2_Open
- removed Q2, Q3: MMBT3904, Package_TO_SOT_SMD:SOT-23, symbol Transistor_BJT:MMBT3904
- removed Q5: AO3400A, Package_TO_SOT_SMD:SOT-23, symbol Transistor_FET:AO3400A
- removed Q6, Q7: AO3401A, Package_TO_SOT_SMD:SOT-23, symbol Transistor_FET:AO3401A
- removed R1, R25, R33, R34, R36, R37, R5: 10k, Resistor_SMD:R_0603_1608Metric, symbol Device:R
- removed R24: 100k, Resistor_SMD:R_0603_1608Metric, symbol Device:R
- removed R28: 4.7k, Resistor_SMD:R_0603_1608Metric, symbol Device:R
- removed R3: 47k, Resistor_SMD:R_0603_1608Metric, symbol Device:R
- removed R30, R31: 5.1k, Resistor_SMD:R_0603_1608Metric, symbol Device:R
- removed R6: 3.9k, Resistor_SMD:R_0603_1608Metric, symbol Device:R
- removed SW1: SW_ENTER, Button_Switch_SMD:SW_Push_1P1T_XKB_TS-1187A, symbol Switch:SW_Push
- removed SW2: SW_BACK, Button_Switch_SMD:SW_Push_1P1T_XKB_TS-1187A, symbol Switch:SW_Push
- removed SW3: SW_DOWN, Button_Switch_SMD:SW_Push_1P1T_XKB_TS-1187A, symbol Switch:SW_Push
- removed SW4: SW_UP, Button_Switch_SMD:SW_Push_1P1T_XKB_TS-1187A, symbol Switch:SW_Push
- removed SW5: SW_ESP_BOOT_MODE, Button_Switch_SMD:SW_Push_1P1T_XKB_TS-1187A, symbol Switch:SW_Push
- removed SW6: SW_ESP_RESET, Button_Switch_SMD:SW_Push_1P1T_XKB_TS-1187A, symbol Switch:SW_Push
- removed SW7: PWR, footprints:SS-12D07-VG 4 NS GA PA, symbol Switch:SW_SPDT
- removed TP11: PSU_EN, TestPoint:TestPoint_Pad_1.0x1.0mm, symbol Connector:TestPoint
- removed TP12: TP_VUSB, TestPoint:TestPoint_Pad_1.0x1.0mm, symbol Connector:TestPoint
- removed TP13: TP_VPSU, TestPoint:TestPoint_Pad_1.0x1.0mm, symbol Connector:TestPoint
- removed TP15: TP_MUX, TestPoint:TestPoint_Pad_1.0x1.0mm, symbol Connector:TestPoint
- removed TP16: ADC_LDO, TestPoint:TestPoint_Pad_1.0x1.0mm, symbol Connector:TestPoint
- removed TP17: TP_ISENSE, TestPoint:TestPoint_Pad_1.0x1.0mm, symbol Connector:TestPoint
- removed TP18: TP_GND, TestPoint:TestPoint_Pad_1.0x1.0mm, symbol Connector:TestPoint
- removed TP19: TP_3V3, TestPoint:TestPoint_Pad_1.0x1.0mm, symbol Connector:TestPoint
- removed TP2: IO40, TestPoint:TestPoint_Pad_1.0x1.0mm, symbol Connector:TestPoint
- removed TP20: TP_SCL, TestPoint:TestPoint_Pad_1.0x1.0mm, symbol Connector:TestPoint
- removed TP21: TP_SDA, TestPoint:TestPoint_Pad_1.0x1.0mm, symbol Connector:TestPoint
- removed TP22: 5V_RAW, TestPoint:TestPoint_Pad_1.0x1.0mm, symbol Connector:TestPoint
- removed TP23: GPS_RST, TestPoint:TestPoint_Pad_1.0x1.0mm, symbol Connector:TestPoint
- removed TP24: B_SENSE, TestPoint:TestPoint_Pad_1.0x1.0mm, symbol Connector:TestPoint
- removed TP25: GPS_TX, TestPoint:TestPoint_Pad_1.0x1.0mm, symbol Connector:TestPoint
- removed TP26: GPS_RX, TestPoint:TestPoint_Pad_1.0x1.0mm, symbol Connector:TestPoint
- removed TP3: IO41, TestPoint:TestPoint_Pad_1.0x1.0mm, symbol Connector:TestPoint
- removed TP4: IO42, TestPoint:TestPoint_Pad_1.0x1.0mm, symbol Connector:TestPoint
- removed TP6: IO4, TestPoint:TestPoint_Pad_1.0x1.0mm, symbol Connector:TestPoint
- removed TP7: I2S_LRCLK, TestPoint:TestPoint_Pad_1.0x1.0mm, symbol Connector:TestPoint
- removed TP8: I2S_BLCK, TestPoint:TestPoint_Pad_1.0x1.0mm, symbol Connector:TestPoint
- removed U1: CP2102N-Axx-xQFN28, Package_DFN_QFN:QFN-28-1EP_5x5mm_P0.5mm_EP3.35x3.35mm, symbol Interface_USB:CP2102N-Axx-xQFN28
- removed U10: MAX98357AETE_T, footprints:MAX98357_QFN50P300X300X80-17N, symbol MAX98357AETE_T:MAX98357AETE_T
- removed U11: RFM95W-915S2, footprints:RFM95W, symbol RF_Module:RFM95W-915S2
- removed U12: YIC31616GMSGG GPS, footprints:YIC31616GMSGG, symbol YIC31616GMSGG:YIC31616GMSGG
- removed U3: TPB4056B2X-ES1R, TPB4056B2X:ES1ESOP-8-F_TPK, symbol TPB4056B2X-ES1R:TPB4056B2X-ES1R
- removed U4: TPS63001DRCR, Package_SON:Texas_DRC0010J_ThermalVias, symbol Regulator_Switching:TPS63001
- removed U6: LM66100DCKR, LMR66100:SC-70-6_Handsoldering, symbol QRET_Buck_PSU:LM66100DCKR
- removed U7: NAU7802SGI, NAU7802SGI:SOI16_NAU7802SGI_NUV, symbol NAU7802SGI:NAU7802SGI
- removed U9: AMS1117-3.3, Package_TO_SOT_SMD:SOT-223-3_TabPin2, symbol Regulator_Linear:AMS1117-3.3
- added C11: 47uF, Capacitor_SMD:C_0805_2012Metric, symbol Device:C
- added C11 (x2), C3 (x3), C4 (x2), C5 (x2): 0.1uF, Capacitor_SMD:C_0603_1608Metric, symbol Device:C
- added C3 (x2), C4 (x4), C5: 10uF, Capacitor_SMD:C_0603_1608Metric, symbol Device:C
- added C3, C4 (x3), C5 (x3): 1uF, Capacitor_SMD:C_0603_1608Metric, symbol Device:C
- added C4: 4.7uF, Capacitor_SMD:C_0603_1608Metric, symbol Device:C
- added C7: 100uF, Capacitor_SMD:CP_Elec_6.3x5.9, symbol Device:C_Polarized
- added D1: INT_PWR_LED (RED), LED_SMD:LED_0805_2012Metric, symbol Device:LED
- added D1: DB_LED (GRN), LED_SMD:LED_0805_2012Metric, symbol Device:LED
- added D4, D7: WS2812B, LED_SMD:LED_WS2812B_PLCC4_5.0x5.0mm_P3.2mm, symbol LED:WS2812B
- added D8: 1N5819WS, Diode_SMD:D_SOD-323_HandSoldering, symbol Diode:1N5817
- added J2: MSD-1-A MicroSD Slot, footprints:MicroSD_MSD-1-A, symbol Connector:Micro_SD_Card_Det1
- added J3: ~, Connector_PinHeader_1.27mm:PinHeader_1x08_P1.27mm_Vertical, symbol E-Paper:Generic_E-Paper_Display
- added J4: USB_C_Female_USB2_Small, footprints:USB_C_DB-108PWB, symbol USB_C:USB_C_Female_USB2_Small
- added J4: 1S Li-Ion Cell, TerminalBlock_TE-Connectivity:TerminalBlock_TE_282834-2_1x02_P2.54mm_Horizontal, symbol Connector:Screw_Terminal_01x02
- added J6: MB_A, Connector_PinSocket_1.27mm:PinSocket_2x02_P1.27mm_Vertical, symbol CONN4_LPPB022NFSS-RC_SUL_SOCKET:LPPB022NFSS-RC
- added J7: MB_B, Connector_PinSocket_1.27mm:PinSocket_2x02_P1.27mm_Vertical, symbol CONN4_LPPB022NFSS-RC_SUL_SOCKET:LPPB022NFSS-RC
- added J8: DB_A, footprints:HPH2-A-04-UA_PINS, symbol CONN4_LPPB022NFSS-RC_SUL_SOCKET:LPPB022NFSS-RC
- added J9: DB_B, footprints:HPH2-A-04-UA_PINS, symbol CONN4_LPPB022NFSS-RC_SUL_SOCKET:LPPB022NFSS-RC
- added JP1: DIO2_EN, Jumper:SolderJumper-2_P1.3mm_Open_RoundedPad1.0x1.5mm, symbol Jumper:SolderJumper_2_Open
- added JP2: Gain, Jumper:SolderJumper-3_P1.3mm_Bridged12_Pad1.0x1.5mm_NumberLabels, symbol Jumper:SolderJumper_3_Bridged12
- added JP4: FastCharge, Jumper:SolderJumper-2_P1.3mm_Open_Pad1.0x1.5mm, symbol Jumper:SolderJumper_2_Open
- added JP5: DB_LED_EN, Jumper:SolderJumper-2_P1.3mm_Bridged_Pad1.0x1.5mm, symbol Jumper:SolderJumper_2_Bridged
- added Q3: AO3401A, Package_TO_SOT_SMD:SOT-23, symbol Transistor_FET:AO3401A
- added Q7: AO3400A, Package_TO_SOT_SMD:SOT-23, symbol Transistor_FET:AO3400A
- added R28: 1k, Resistor_SMD:R_0603_1608Metric, symbol Device:R
- added R28: 5.1k, Resistor_SMD:R_0603_1608Metric, symbol Device:R
- added R39: 510, Resistor_SMD:R_0603_1608Metric, symbol Device:R
- added R5: 10k, Resistor_SMD:R_0603_1608Metric, symbol Device:R
- added R5: 1.8k, Resistor_SMD:R_0603_1608Metric, symbol Device:R
- added SW1: PWR, footprints:SS-12D07-VG 4 NS GA PA, symbol Switch:SW_SPDT
- added SW2: SW_ESP_BOOT_MODE, Button_Switch_SMD:SW_Push_1P1T_XKB_TS-1187A, symbol Switch:SW_Push
- added SW2: SW_ESP_RESET, Button_Switch_SMD:SW_Push_1P1T_XKB_TS-1187A, symbol Switch:SW_Push
- added SW2: SW_ENTER, Button_Switch_SMD:SW_Push_1P1T_XKB_TS-1187A, symbol Switch:SW_Push
- added SW2: SW_DOWN, Button_Switch_SMD:SW_Push_1P1T_XKB_TS-1187A, symbol Switch:SW_Push
- added SW2: SW_UP, Button_Switch_SMD:SW_Push_1P1T_XKB_TS-1187A, symbol Switch:SW_Push
- added SW2: SW_BACK, Button_Switch_SMD:SW_Push_1P1T_XKB_TS-1187A, symbol Switch:SW_Push
- added TP2: CHRG_STAT, TestPoint:TestPoint_Pad_1.0x1.0mm, symbol Connector:TestPoint
- added TP2: TP_VUSB, TestPoint:TestPoint_Pad_1.0x1.0mm, symbol Connector:TestPoint
- added TP4: TP_BTN, TestPoint:TestPoint_Pad_1.0x1.0mm, symbol Connector:TestPoint
- added TP4: TP_MUX, TestPoint:TestPoint_Pad_1.0x1.0mm, symbol Connector:TestPoint
- added TP8: GPS_RX, TestPoint:TestPoint_Pad_1.0x1.0mm, symbol Connector:TestPoint
- added TP8: IO40, TestPoint:TestPoint_Pad_1.0x1.0mm, symbol Connector:TestPoint
- added TP8: GPS_RST, TestPoint:TestPoint_Pad_1.0x1.0mm, symbol Connector:TestPoint
- added TP8: IO42, TestPoint:TestPoint_Pad_1.0x1.0mm, symbol Connector:TestPoint
- added TP8: GPS_TX, TestPoint:TestPoint_Pad_1.0x1.0mm, symbol Connector:TestPoint
- added TP8: I2S_LRCLK, TestPoint:TestPoint_Pad_1.0x1.0mm, symbol Connector:TestPoint
- added TP8: IO4, TestPoint:TestPoint_Pad_1.0x1.0mm, symbol Connector:TestPoint
- added TP8: 5V_RAW, TestPoint:TestPoint_Pad_1.0x1.0mm, symbol Connector:TestPoint
- added TP8: TP_ISENSE, TestPoint:TestPoint_Pad_1.0x1.0mm, symbol Connector:TestPoint
- added TP8: I2S_BLCK, TestPoint:TestPoint_Pad_1.0x1.0mm, symbol Connector:TestPoint
- added TP8: IO41, TestPoint:TestPoint_Pad_1.0x1.0mm, symbol Connector:TestPoint
- added TP8: I2S_DIN, TestPoint:TestPoint_Pad_1.0x1.0mm, symbol Connector:TestPoint
- added U1: RFM95W-915S2, footprints:RFM95W, symbol RF_Module:RFM95W-915S2
- added U10: TPB4056B2X-ES1R, TPB4056B2X:ES1ESOP-8-F_TPK, symbol TPB4056B2X-ES1R:TPB4056B2X-ES1R
- added U12: AMS1117-3.3, Package_TO_SOT_SMD:SOT-223-3_TabPin2, symbol Regulator_Linear:AMS1117-3.3
- added U4: LM66100DCKR, LMR66100:SC-70-6_Handsoldering, symbol QRET_Buck_PSU:LM66100DCKR
- added U7: MAX98357AETE_T, footprints:MAX98357_QFN50P300X300X80-17N, symbol MAX98357AETE_T:MAX98357AETE_T
- added U8: TPS63001DRCR, Package_SON:Texas_DRC0010J_ThermalVias, symbol Regulator_Switching:TPS63001
- added U9: YIC31616GMSGG GPS, footprints:YIC31616GMSGG, symbol YIC31616GMSGG:YIC31616GMSGG
- C1: value 1uF -> 10uF; LCSC C15849 -> C96446
- C13: JLCPCB (none) -> C15849; LCSC C15849 -> (none)
- C19: value 100uF -> 330mF; footprint Capacitor_SMD:CP_Elec_6.3x5.9 -> footprints:CB5R5334HF-ZJP; Digikey 732-8419-1-ND -> 4688-CB5R5334HF-ZJP-ND; Model (none) -> CB5R5334HF-ZJP
- JP3: value ADC_REFP -> SPK_DIN; now left out of the parts list
- R10: value 2k -> 51k; LCSC C22975 -> C23196
- R11: value 1k -> 10k; LCSC C21190 -> C25804
- R13: value 51k -> 1k; LCSC C23196 -> C21190
- R14: value 2.4k -> 2k; LCSC C22940 -> C22975
- R15: value 1k -> 5.6k; LCSC C21190 -> C23189
- R17: value 10k -> 20k; LCSC C25804 -> C4184
- R19: value 510 -> 100R; JLCPCB (none) -> C22775; LCSC C23193 -> (none)
- R2: value 22k -> 10k; LCSC C31850 -> C25804
- R22: value 100k -> 10k; LCSC C25803 -> C25804
- R23: value 51k -> 10k; LCSC C23196 -> C25804
- R26: value 1.8k -> 10k; LCSC C4177 -> C25804
- R27: value 4.7k -> 10k; LCSC C23162 -> C25804
- R29: value 1.5k -> 5.1k; LCSC C22843 -> C23186
- R35: value 10k -> 100; LCSC C25804 -> C22775
- R38: value 10k -> 100k; LCSC C25804 -> C25803
- R4: value 1k -> 100k; LCSC C21190 -> C25803
- R7: value 100 -> 2.4k; LCSC C22775 -> C22940
- R8: value 100k -> 3.9k; LCSC C25803 -> C23018
- R9: value 5.6k -> 100k; LCSC C23189 -> C25803
- TP1: value IO39 -> TP_VPSU
- TP10: value TP_BTN -> TP_3V3
- TP14: value CHRG_STAT -> BKP; footprint TestPoint:TestPoint_Pad_1.0x1.0mm -> TestPoint:TestPoint_Pad_1.5x1.5mm
- TP5: value IO45 -> B_SENSE
- TP9: value I2S_DIN -> TP_GND
Connections:
- net DTR is gone; now on net BATT_SENSE: R16.1
- net I2C_SDA is gone; now on net RESET_RF: U2.25 (GPIO48/SPICLK_N/SUBSPICLK_N_DIFF)
- net RTS is gone; now on net BATT_SENSE: R17.2
- net UART0_RX is gone; now on net UART1_GPS_RX: U2.36 (U0RXD/GPIO44/CLK_OUT2)
- net UART0_TX is gone; now on net UART1_GPS_TX: U2.37 (U0TXD/GPIO43/CLK_OUT1)
- net +3.3V: now also C13.1, R11.1, R2.2, R20.1, R21.1, R22.1, R23.1, TP10.1, C11.1, C11.1, C3.1, C3.1, C4.2, C4.2, C5.1, C5.1, D8.2 (A), J2.4 (VDD), J3.1 (VCC), J6.4, J7.4, JP2.3 (B), R5.2, U1.13 (3.3V), U7.7 (VDD), U7.8 (VDD__1), U9.4 (VCC); no longer JP3.1 (A), R20.2, R26.2, R29.2, R35.1
- net +3.3VA: now also C4.2, C4.2, D4.1 (VDD), D7.1 (VDD), J8.4, J9.4, SW2.1, SW2.1, SW2.1, SW2.1
- net +5V: now also C1.1, C5.1, C5.2, Q3.3 (D), U10.4 (VIN), U10.8 (CE), U12.3 (VI); no longer Q1.1 (G), R8.1
- net +BATT: now also Q1.2 (S), R17.1, R35.1, R4.1, C4.1, U8.5 (VIN); no longer R7.1
- net 5V_OFF: now also R38.1, U2.24 (GPIO47/SPICLK_P/SUBSPICLK_P_DIFF), R39.1; no longer R18.1, R19.1, U2.15 (GPIO3/TOUCH3/ADC1_CH2)
- net 5V_RAW: now also R10.1, R9.1, C4.2, J4.A4 (VBUS), J4.A9 (VBUS), J4.B4 (VBUS), J4.B9 (VBUS), Q3.2 (S), TP8.1; no longer R2.2, R22.1, R23.1
- net ARGB_DATA: now also J7.3, JP5.1 (A)
- net ARGB_DATA_DB: now also J9.3
- net BATT_SENSE: now also TP5.1, U2.15 (GPIO3/TOUCH3/ADC1_CH2); no longer R38.1
- net BUTTONS: now also J7.1
- net BUTTONS_DB: now also R13.2, R14.1, J9.1, R28.2, TP4.1; no longer R10.1, R11.2, R9.2, TP10.1
- net CHRG_STAT: now also R26.2, R27.1, TP2.1, U10.7 (CHRG); no longer R20.1, R21.2, TP14.1
- net CLK_SDMMC: now also R23.2, J2.5 (CLK)
- net CMD_SDMMC: now also R21.2, U2.30 (SPIDQS/GPIO37/FSPIQ/SUBSPIQ), J2.3 (CMD); no longer R32.2, U2.28 (SPIIO6/GPIO35/FSPID/SUBSPID)
- net CS_EINK: now also J3.5 (CS)
- net CS_RF: now also U1.5 (NSS)
- net CURR_SENSE: now also U2.7 (GPIO7/TOUCH7/ADC1_CH6), TP8.1
- net D0_SDMMC: now also R22.2, U2.28 (SPIIO6/GPIO35/FSPID/SUBSPID), J2.7 (DAT0); no longer U2.30 (SPIDQS/GPIO37/FSPIQ/SUBSPIQ)
- net DIO0_RF: now also U1.14 (DIO0)
- net DIO1_RF: now also U1.15 (DIO1)
- net DIO2_RF: now also JP1.2 (B), TP8.1
- net EINK_BUSY: now also J3.8 (BUSY), TP8.1
- net EINK_DC: now also J3.6 (DC)
- net ESP32_EN: now also R32.2, C3.2, C3.2, SW2.2; no longer C1.2
- net GND: now also C1.2, Q1.1 (G), R16.2, R29.2, R7.1, TP9.1, C11.2, C11.2, C11.2, C3.1, C3.1, C3.1, C3.2, C3.2, C3.2, C4.1, C4.1, C4.1, C4.2, C4.2, C4.2, C4.2, C4.2, C5.1, C5.1, C5.2, C5.2, C5.2, C5.2, C7.2, D1.1 (K), D1.1 (K), J2.10 (SHIELD), J2.6 (VSS), J3.2 (GND), J4.1 (Pin_1), J4.A1 (GND), J4.A12 (GND), J4.B1 (GND), J4.B12 (GND), J6.2, J7.2, JP2.1 (A), Q7.2 (S), R28.2, SW2.1, SW2.1, U1.1 (GND), U1.10 (GND), U1.8 (GND), U10.1 (TEMP), U10.3 (GND), U10.9 (GND), U12.1 (GND), U4.2 (GND), U4.5 (ST), U7.11 (GND__1), U7.15 (GND__2), U7.17 (EP), U7.3 (GND), U8.11 (PGND), U8.3 (PGND), U8.9 (GND), U9.12 (GND), U9.3 (GND); no longer C1.1, R13.1, R14.1, R18.2, R4.2
- net GND2: now also C4.1, C4.1, D4.3 (VSS), D7.3 (VSS), J8.2, J9.2, R28.1; no longer R15.1
- net GPIO0: now also C3.2, SW2.2
- net GPS_RST: now also R11.2, TP8.1, U9.10 (RESET)
- net I2S_BCLK_SPK: now also TP8.1, U7.16 (BCLK)
- net I2S_DIN_SPK: now also JP3.2 (B), TP8.1; no longer TP9.1
- net I2S_LRCLK_SPK: now also TP8.1, U7.14 (LRCLK)
- net LA: now also U8.2 (L2)
- net LB: now also U8.4 (L1)
- net MISO_EINK: now also TP8.1
- net MISO_RF: now also U1.2 (MISO)
- net MOSI_EINK: now also J3.3 (DIN)
- net MOSI_RF: now also U1.3 (MOSI)
- net RAW_BATT: now also C5.2, J4.2 (Pin_2), SW1.2 (B), U10.5 (BAT)
- net RESET_EINK: now also J3.7 (RST)
- net RESET_RF: now also R2.1, U1.6 (RESET); no longer U2.7 (GPIO7/TOUCH7/ADC1_CH6)
- net SCK_EINK: now also J3.4 (CLK)
- net SCK_RF: now also U1.4 (SCK)
- net SPK_ON: now also R18.1, TP8.1
- net UART1_GPS_RX: now also TP8.1, U9.2 (TXD); no longer U2.13 (GPIO19/U1RTS/ADC2_CH8/CLK_OUT2/USB_D-)
- net UART1_GPS_TX: now also TP8.1, U9.1 (RXD); no longer U2.14 (GPIO20/U1CTS/ADC2_CH9/CLK_OUT1/USB_D+)
- net USB_D+: now also U2.14 (GPIO20/U1CTS/ADC2_CH9/CLK_OUT1/USB_D+), J4.A6 (D+), J4.B6 (D+); no longer R29.1
- net USB_D-: now also U2.13 (GPIO19/U1RTS/ADC2_CH8/CLK_OUT2/USB_D-), J4.A7 (D-), J4.B7 (D-)
- net V_MUX: now also C11.1, C7.1, TP4.1, U4.3 (*CE), U4.6 (VOUT); no longer C19.1
- net V_PSU: now also TP1.1, U5.1 (VIN), C4.1, C4.1, C5.1, U8.1 (VOUT), U8.10 (FB); no longer C13.1
- net V_REGUSB: now also C3.1, C4.1, TP2.1, U12.2 (VO), U4.1 (VIN); no longer U5.1 (VIN)
- net at R14.2: now also SW2.2
- net at R10.2: now also Q4.3 (D), Q3.1 (G)
- net at U2.32 (MTCK/GPIO39/CLK_OUT3/SUBSPICS1): no longer TP1.1
- net at D6.2 (DOUT): now also D7.4 (DIN)
- net at AE1.1 (A): now also U1.9 (ANT)
- net at D5.4 (DIN): now also D4.2 (DOUT)
- net at R26.1: now also U10.6 (STBY)
- net at Q4.1 (G): now also R9.2, Q7.3 (D); no longer R19.2
- net at R7.2: now also JP4.2 (B), U10.2 (PROG); no longer Q1.2 (S)
- net at Q1.3 (D): now also SW1.1 (A); no longer R13.2
- net at R35.2: now also C4.1, U8.7 (PS/SYNC), U8.8 (VINA)
- net at U2.26 (GPIO45): no longer TP5.1
- net at R12.1: now also SW2.2
- net at D1.2 (DOUT): now also D4.4 (DIN)
- net at J5.1 (Pin_1): now also U7.10 (OUTN)
- net at J5.2 (Pin_2): now also U7.9 (OUTP)
- removed net I2C_SCL: R27.1, U2.24 (GPIO47/SPICLK_P/SUBSPICLK_P_DIFF)
- new net: D8.1 (K), R19.1
- new net: JP5.2 (B), R5.2
- new net: D1.2 (A), R5.1 (x2)
- new net: J4.A5 (CC1), R29.1
- new net: R4.2, U8.6 (EN)
- new net: J2.2 (DAT3/CD), R20.2
- new net: J4.B5 (CC2), R28.1
- new net: JP4.1 (A), R8.1
- new net: JP1.1 (A), U1.16 (DIO2)
- new net: R15.1, SW2.2
- new net: Q7.1 (G), R39.2
- new net: R13.1, SW2.2
- new net: R18.2, U7.4 (SD_MODE)
- new net: JP3.1 (A), U7.1 (DIN)
- new net: JP2.2 (C), U7.2 (GAIN_SLOT)
- new net GPS_BCKP: C19.1, R19.2, TP14.1, U9.5 (V_BCKP)
- no-connect marks 42 -> 22
Other:
- note added: "ESP32 DB Buttons"
- note added: "GPS + Backup Capcitor"
- note added: "V=3.3V, R=100, I(max)=33mA Usable voltage range: 1.65V - 3.60V 1N5819 V(fw) trends towards 200mV -> 3.1V max charge"
- note removed: "ESP32 Auto-Programmer & DB Buttons"
- note removed: "External I2C ADC was used simply to save on GPIO pins in case there is an error on the PCB."
- note removed: "GPS"
- note removed: "I2C ADDRESS: >0x2A (fixed)"
- note removed: "I2C ADDRESS: >0x48 (A2,1,0=0)"
- note removed: "Power Monitoring ADC"
- note removed: "Temperature Sensor (I2C)"
- note removed: "USB-UART Bridge"
- note removed: "[UPDATE] SHOULD BE PULLUP !!!"
- title: (none) -> Kuhglocke Ground Station

Commit message: added silkscreen for eink pins
Other:
- company: (none) -> Queen's Rocket Engineering Team
- title: Kuhglocke Ground Station -> QRET 25-26 SRAD Handheld Ground Station
Changed lines of the file:
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@@
 	(paper "B")
 	(title_block
-		(title "Kuhglocke Ground Station")
+		(title "QRET 25-26 SRAD Handheld Ground Station")
 		(date "2024-05-29")
-		(rev "V1.0")
+		(rev "V0.2.0")
+		(company "Queen's Rocket Engineering Team")
+		(comment 1 "Contributors: Kennan Bays, Tristan Alderson, Ethan Toste")
 		(comment 3 "GRID: 1.27mm")
-		(comment 4 "Contributors: Kennan Bays")
 	)
 	(junction
